Commit message: data folder restructured and readme updated

File: data/raw/urdf/robots_h2_description_H2.urdf (robot description, URDF)
Before this commit: robot H2, 34 links, 33 joints
Links:
- added link camera
- added link imu_in_pelvis
- added link imu_in_torso
- link head_pitch_link: geometry visual mesh filename=meshes/head_pitch_link.stl
- link head_yaw_link: geometry collision mesh filename=meshes/head_yaw_link.stl; visual mesh filename=meshes/head_yaw_link.stl
- link left_ankle_pitch_link: geometry collision mesh filename=meshes/left_ankle_pitch_link.stl; visual mesh filename=meshes/left_ankle_pitch_link.stl
- link left_ankle_roll_link: geometry visual mesh filename=meshes/left_ankle_roll_link.stl
- link left_elbow_link: geometry collision mesh filename=meshes/left_elbow_link.stl; visual mesh filename=meshes/left_elbow_link.stl
- link left_hand_link: geometry collision mesh filename=meshes/left_hand_link.stl; visual mesh filename=meshes/left_hand_link.stl
- link left_hip_pitch_link: geometry visual mesh filename=meshes/left_hip_pitch_link.stl
- link left_hip_roll_link: geometry collision sphere radius=0.05; visual mesh filename=meshes/left_hip_roll_link.stl
- link left_hip_yaw_link: geometry collision mesh filename=meshes/left_hip_yaw_link.stl; visual mesh filename=meshes/left_hip_yaw_link.stl
- link left_knee_link: geometry collision cylinder length=0.35 radius=0.025; visual mesh filename=meshes/left_knee_link.stl
- link left_shoulder_pitch_link: geometry collision mesh filename=meshes/left_shoulder_pitch_link.stl; visual mesh filename=meshes/left_shoulder_pitch_link.stl
- link left_shoulder_roll_link: geometry collision mesh filename=meshes/left_shoulder_roll_link.stl; visual mesh filename=meshes/left_shoulder_roll_link.stl
- link left_shoulder_yaw_link: geometry collision mesh filename=meshes/left_shoulder_yaw_link.stl; visual mesh filename=meshes/left_shoulder_yaw_link.stl
- link left_wrist_pitch_link: geometry visual mesh filename=meshes/left_wrist_pitch_link.stl
- link left_wrist_roll_link: geometry visual mesh filename=meshes/left_wrist_roll_link.stl
- link left_wrist_yaw_link: geometry collision mesh filename=meshes/left_wrist_yaw_link.stl; visual mesh filename=meshes/left_wrist_yaw_link.stl
- link pelvis: geometry collision mesh filename=meshes/pelvis.stl; visual mesh filename=meshes/pelvis.stl
- link right_ankle_pitch_link: geometry collision mesh filename=meshes/right_ankle_pitch_link.stl; visual mesh filename=meshes/right_ankle_pitch_link.stl
- link right_ankle_roll_link: geometry visual mesh filename=meshes/right_ankle_roll_link.stl
- link right_elbow_link: geometry collision mesh filename=meshes/right_elbow_link.stl; visual mesh filename=meshes/right_elbow_link.stl
- link right_hand_link: geometry collision mesh filename=meshes/right_hand_link.stl; visual mesh filename=meshes/right_hand_link.stl
- link right_hip_pitch_link: geometry visual mesh filename=meshes/right_hip_pitch_link.stl
- link right_hip_roll_link: geometry collision sphere radius=0.05; visual mesh filename=meshes/right_hip_roll_link.stl
- link right_hip_yaw_link: geometry collision mesh filename=meshes/right_hip_yaw_link.stl; visual mesh filename=meshes/right_hip_yaw_link.stl
- link right_knee_link: geometry collision cylinder length=0.35 radius=0.025; visual mesh filename=meshes/right_knee_link.stl
- link right_shoulder_pitch_link: geometry collision mesh filename=meshes/right_shoulder_pitch_link.stl; visual mesh filename=meshes/right_shoulder_pitch_link.stl
- link right_shoulder_roll_link: geometry collision mesh filename=meshes/right_shoulder_roll_link.stl; visual mesh filename=meshes/right_shoulder_roll_link.stl
- link right_shoulder_yaw_link: geometry collision mesh filename=meshes/right_shoulder_yaw_link.stl; visual mesh filename=meshes/right_shoulder_yaw_link.stl
- link right_wrist_pitch_link: geometry visual mesh filename=meshes/right_wrist_pitch_link.stl
- link right_wrist_roll_link: geometry visual mesh filename=meshes/right_wrist_roll_link.stl
- link right_wrist_yaw_link: geometry collision mesh filename=meshes/right_wrist_yaw_link.stl; visual mesh filename=meshes/right_wrist_yaw_link.stl
- link torso_link: geometry collision mesh filename=meshes/torso_link.stl; visual mesh filename=meshes/torso_link.stl
- link waist_roll_link: geometry visual mesh filename=meshes/waist_roll_link.stl
- link waist_yaw_link: geometry visual mesh filename=meshes/waist_yaw_link.stl
Joints:
- added joint camera: type fixed, parent head_yaw_link, child camera, origin xyz=0.08667 0.03 0.0099 rpy=0 0 0
- added joint imu_in_pelvis_joint: type fixed, parent pelvis, child imu_in_pelvis, origin xyz=-0.055 0 -0.0589 rpy=0 0 0
- added joint imu_in_torso_joint: type fixed, parent torso_link, child imu_in_torso, origin xyz=-0.06382 -0.06538 0.29588 rpy=0 0 0

File: data/raw/urdf/robots_h2_description_H2_dae.urdf (robot description, URDF)
Before this commit: robot H2, 34 links, 33 joints
Links:
- added link camera
- added link imu_in_pelvis
- added link imu_in_torso
- link head_pitch_link: geometry visual mesh filename=meshes/head_pitch_link.dae
- link head_yaw_link: geometry collision mesh filename=meshes/head_yaw_link.stl; visual mesh filename=meshes/head_yaw_link.dae
- link left_ankle_pitch_link: geometry collision mesh filename=meshes/left_ankle_pitch_link.stl; visual mesh filename=meshes/left_ankle_pitch_link.dae
- link left_ankle_roll_link: geometry visual mesh filename=meshes/left_ankle_roll_link.dae
- link left_elbow_link: geometry collision mesh filename=meshes/left_elbow_link.stl; visual mesh filename=meshes/left_elbow_link.dae
- link left_hand_link: geometry collision mesh filename=meshes/left_hand_link.stl; visual mesh filename=meshes/left_hand_link.dae
- link left_hip_pitch_link: geometry visual mesh filename=meshes/left_hip_pitch_link.dae
- link left_hip_roll_link: geometry collision sphere radius=0.05; visual mesh filename=meshes/left_hip_roll_link.dae
- link left_hip_yaw_link: geometry collision mesh filename=meshes/left_hip_yaw_link.stl; visual mesh filename=meshes/left_hip_yaw_link.dae
- link left_knee_link: geometry collision cylinder length=0.35 radius=0.025; visual mesh filename=meshes/left_knee_link.dae
- link left_shoulder_pitch_link: geometry collision mesh filename=meshes/left_shoulder_pitch_link.stl; visual mesh filename=meshes/left_shoulder_pitch_link.dae
- link left_shoulder_roll_link: geometry collision mesh filename=meshes/left_shoulder_roll_link.stl; visual mesh filename=meshes/left_shoulder_roll_link.dae
- link left_shoulder_yaw_link: geometry collision mesh filename=meshes/left_shoulder_yaw_link.stl; visual mesh filename=meshes/left_shoulder_yaw_link.dae
- link left_wrist_pitch_link: geometry visual mesh filename=meshes/left_wrist_pitch_link.dae
- link left_wrist_roll_link: geometry visual mesh filename=meshes/left_wrist_roll_link.dae
- link left_wrist_yaw_link: geometry collision mesh filename=meshes/left_wrist_yaw_link.stl; visual mesh filename=meshes/left_wrist_yaw_link.dae
- link pelvis: geometry collision mesh filename=meshes/pelvis.stl; visual mesh filename=meshes/pelvis.dae
- link right_ankle_pitch_link: geometry collision mesh filename=meshes/right_ankle_pitch_link.stl; visual mesh filename=meshes/right_ankle_pitch_link.dae
- link right_ankle_roll_link: geometry visual mesh filename=meshes/right_ankle_roll_link.dae
- link right_elbow_link: geometry collision mesh filename=meshes/right_elbow_link.stl; visual mesh filename=meshes/right_elbow_link.dae
- link right_hand_link: geometry collision mesh filename=meshes/right_hand_link.stl; visual mesh filename=meshes/right_hand_link.dae
- link right_hip_pitch_link: geometry visual mesh filename=meshes/right_hip_pitch_link.dae
- link right_hip_roll_link: geometry collision sphere radius=0.05; visual mesh filename=meshes/right_hip_roll_link.dae
- link right_hip_yaw_link: geometry collision mesh filename=meshes/right_hip_yaw_link.stl; visual mesh filename=meshes/right_hip_yaw_link.dae
- link right_knee_link: geometry collision cylinder length=0.35 radius=0.025; visual mesh filename=meshes/right_knee_link.dae
- link right_shoulder_pitch_link: geometry collision mesh filename=meshes/right_shoulder_pitch_link.stl; visual mesh filename=meshes/right_shoulder_pitch_link.dae
- link right_shoulder_roll_link: geometry collision mesh filename=meshes/right_shoulder_roll_link.stl; visual mesh filename=meshes/right_shoulder_roll_link.dae
- link right_shoulder_yaw_link: geometry collision mesh filename=meshes/right_shoulder_yaw_link.stl; visual mesh filename=meshes/right_shoulder_yaw_link.dae
- link right_wrist_pitch_link: geometry visual mesh filename=meshes/right_wrist_pitch_link.dae
- link right_wrist_roll_link: geometry visual mesh filename=meshes/right_wrist_roll_link.dae
- link right_wrist_yaw_link: geometry collision mesh filename=meshes/right_wrist_yaw_link.stl; visual mesh filename=meshes/right_wrist_yaw_link.dae
- link torso_link: geometry collision mesh filename=meshes/torso_link.stl; visual mesh filename=meshes/torso_link.dae
- link waist_roll_link: geometry visual mesh filename=meshes/waist_roll_link.dae
- link waist_yaw_link: geometry visual mesh filename=meshes/waist_yaw_link.dae
Joints:
- added joint camera: type fixed, parent head_yaw_link, child camera, origin xyz=0.08667 0.03 0.0099 rpy=0 0 0
- added joint imu_in_pelvis_joint: type fixed, parent pelvis, child imu_in_pelvis, origin xyz=-0.055 0 -0.0589 rpy=0 0 0
- added joint imu_in_torso_joint: type fixed, parent torso_link, child imu_in_torso, origin xyz=-0.06382 -0.06538 0.29588 rpy=0 0 0
