Commit message: cat 3 almost finish

File: data/cat3/raw/eve_r3/source.urdf (robot description, URDF)
Before this commit: robot eve_r3, 96 links, 95 joints
Joints:
- joint j_ankle_x: limit lower=-0.523599 upper=0.523599 effort=1e30 velocity=1e30 -> lower=-0.523599 upper=0.523599 effort=-1.0 velocity=-1.0
- joint j_ankle_y: limit lower=-1.57 upper=0.174533 effort=1e30 velocity=1e30 -> lower=-1.57 upper=0.174533 effort=-1.0 velocity=-1.0
- joint j_hip_x: limit lower=-0.523599 upper=0.523599 effort=1e30 velocity=1e30 -> lower=-0.523599 upper=0.523599 effort=-1.0 velocity=-1.0
- joint j_hip_y: limit lower=-1.57 upper=0.174533 effort=1e30 velocity=1e30 -> lower=-1.57 upper=0.174533 effort=-1.0 velocity=-1.0
- joint j_hip_z: limit lower=-1.0472 upper=1.0472 effort=1e30 velocity=1e30 -> lower=-1.0472 upper=1.0472 effort=-1.0 velocity=-1.0
- joint j_knee_y: limit lower=0.0 upper=2.583 effort=1e30 velocity=1e30 -> lower=0.0 upper=2.583 effort=-1.0 velocity=-1.0
- joint j_l_elbow_y: limit lower=-2.18166 upper=0.0 effort=1e30 velocity=1e30 -> lower=-2.18166 upper=0.0 effort=-1.0 velocity=-1.0
- joint j_l_elbow_z: limit lower=-1.5708 upper=0.7854 effort=1e30 velocity=1e30 -> lower=-1.5708 upper=0.7854 effort=-1.0 velocity=-1.0
- joint j_l_shoulder_x: limit lower=-0.0872665 upper=2.0943951 effort=1e30 velocity=1e30 -> lower=-0.0872665 upper=2.0943951 effort=-1.0 velocity=-1.0
- joint j_l_shoulder_y: limit lower=-2.4240878 upper=0.981049573 effort=1e30 velocity=1e30 -> lower=-2.4240878 upper=0.981049573 effort=-1.0 velocity=-1.0
- joint j_l_shoulder_z: limit lower=-1.4660761 upper=0.5410525 effort=1e30 velocity=1e30 -> lower=-1.4660761 upper=0.5410525 effort=-1.0 velocity=-1.0
- joint j_l_wheel_y: limit lower=-1.0E16 upper=1.0E16 effort=1e30 velocity=1e30 -> lower=-1.0E16 upper=1.0E16 effort=-1.0 velocity=-1.0
- joint j_l_wrist_x: limit lower=-1.5708 upper=0.523599 effort=1e30 velocity=1e30 -> lower=-1.5708 upper=0.523599 effort=-1.0 velocity=-1.0
- joint j_l_wrist_y: limit lower=-0.785398 upper=0.785398 effort=1e30 velocity=1e30 -> lower=-0.785398 upper=0.785398 effort=-1.0 velocity=-1.0
- joint j_neck_y: limit lower=-0.335 upper=0.506 effort=1e30 velocity=1e30 -> lower=-0.335 upper=0.506 effort=-1.0 velocity=-1.0
- joint j_r_elbow_y: limit lower=-2.18166 upper=0.0 effort=1e30 velocity=1e30 -> lower=-2.18166 upper=0.0 effort=-1.0 velocity=-1.0
- joint j_r_elbow_z: limit lower=-0.7854 upper=1.5708 effort=1e30 velocity=1e30 -> lower=-0.7854 upper=1.5708 effort=-1.0 velocity=-1.0
- joint j_r_shoulder_x: limit lower=-2.0943951 upper=0.0872665 effort=1e30 velocity=1e30 -> lower=-2.0943951 upper=0.0872665 effort=-1.0 velocity=-1.0
- joint j_r_shoulder_y: limit lower=-2.4240878 upper=0.981049573 effort=1e30 velocity=1e30 -> lower=-2.4240878 upper=0.981049573 effort=-1.0 velocity=-1.0
- joint j_r_shoulder_z: limit lower=-0.5410525 upper=1.4660761 effort=1e30 velocity=1e30 -> lower=-0.5410525 upper=1.4660761 effort=-1.0 velocity=-1.0
- joint j_r_wheel_y: limit lower=-1.0E16 upper=1.0E16 effort=1e30 velocity=1e30 -> lower=-1.0E16 upper=1.0E16 effort=-1.0 velocity=-1.0
- joint j_r_wrist_x: limit lower=-0.523599 upper=1.5708 effort=1e30 velocity=1e30 -> lower=-0.523599 upper=1.5708 effort=-1.0 velocity=-1.0
- joint j_r_wrist_y: limit lower=-0.785398 upper=0.785398 effort=1e30 velocity=1e30 -> lower=-0.785398 upper=0.785398 effort=-1.0 velocity=-1.0
