Commit message: cat3 almost finish, just need the use of an OCR for specific PDF

File: data/cat3/raw/urdf/xarm6/source.urdf (robot description, URDF)
Before this commit: robot UF_ROBOT, 10 links, 9 joints
Links:
- removed link link7
- link link1: mass 2.382 -> 2.3814; geometry collision mesh filename=package://xarm_description/meshes/xarm6/visual/link1.stl; visual mesh filename=package://xarm_description/meshes/xarm6/visual/link1.stl
- link link2: mass 1.869 -> 2.2675; geometry collision mesh filename=package://xarm_description/meshes/xarm6/visual/link2.stl; visual mesh filename=package://xarm_description/meshes/xarm6/visual/link2.stl
- link link3: mass 1.6383 -> 1.875; geometry collision mesh filename=package://xarm_description/meshes/xarm6/visual/link3.stl; visual mesh filename=package://xarm_description/meshes/xarm6/visual/link3.stl
- link link4: mass 1.7269 -> 1.3192; geometry collision mesh filename=package://xarm_description/meshes/xarm6/visual/link4.stl; visual mesh filename=package://xarm_description/meshes/xarm6/visual/link4.stl
- link link5: mass 1.3203 -> 1.33854; geometry collision mesh filename=package://xarm_description/meshes/xarm6/visual/link5.stl; visual mesh filename=package://xarm_description/meshes/xarm6/visual/link5.stl
- link link6: mass 1.325 -> 0.17; geometry collision mesh filename=package://xarm_description/meshes/end_tool/collision/end_to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; visual mesh filename=package://xarm_description/meshes/xarm6/visual/link6.stl
- link link_base: mass 0.88556 -> 2.7; geometry collision mesh filename=package://xarm_description/meshes/xarm6/visual/link_base.stl; visual mesh filename=package://xarm_description/meshes/xarm6/visual/link_base.stl
Joints:
- removed joint joint7
- joint joint1: limit lower=-6.283185307179586 upper=6.283185307179586 effort=50 velocity=3.14 -> lower=-6.283185307179586 upper=6.283185307179586 effort=50.0 velocity=3.14
- joint joint2: limit lower=-2.059 upper=2.0944 effort=50 velocity=3.14 -> lower=-2.059 upper=2.0944 effort=50.0 velocity=3.14
- joint joint3: limit lower=-6.283185307179586 upper=6.283185307179586 effort=30 velocity=3.14 -> lower=-3.927 upper=0.19198 effort=32.0 velocity=3.14; origin xyz=0 -0.293 0 rpy=1.5708 0 0 -> xyz=0.0535 -0.2845 0 rpy=0 0 0
- joint joint4: limit lower=-0.19198 upper=3.927 effort=30 velocity=3.14 -> lower=-6.283185307179586 upper=6.283185307179586 effort=32.0 velocity=3.14; origin xyz=0.0525 0 0 rpy=1.5708 0 0 -> xyz=0.0775 0.3425 0 rpy=-1.5708 0 0
- joint joint5: limit lower=-6.283185307179586 upper=6.283185307179586 effort=30 velocity=3.14 -> lower=-1.69297 upper=3.141592653589793 effort=32.0 velocity=3.14; origin xyz=0.0775 -0.3425 0 rpy=1.5708 0 0 -> xyz=0 0 0 rpy=1.5708 0 0
- joint joint6: limit lower=-1.69297 upper=3.141592653589793 effort=20 velocity=3.14 -> lower=-6.283185307179586 upper=6.283185307179586 effort=20.0 velocity=3.14; origin xyz=0 0 0 rpy=1.5708 0 0 -> xyz=0.076 0.097 0 rpy=-1.5708 0 0
- joint joint_eef: parent link7 -> link6

File: data/cat3/raw/urdf/xarm7/source.urdf (robot description, URDF)
Before this commit: robot UF_ROBOT, 9 links, 8 joints
Links:
- added link link7, mass 0.17; collision mesh filename=package://xarm_description/meshes/end_tool/collision/end_to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; visual mesh filename=package://xarm_description/meshes/xarm7/visual/link7.stl
- link link1: mass 2.3814 -> 2.382; geometry collision mesh filename=package://xarm_description/meshes/xarm7/visual/link1.stl; visual mesh filename=package://xarm_description/meshes/xarm7/visual/link1.stl
- link link2: mass 2.2675 -> 1.869; geometry collision mesh filename=package://xarm_description/meshes/xarm7/visual/link2.stl; visual mesh filename=package://xarm_description/meshes/xarm7/visual/link2.stl
- link link3: mass 1.875 -> 1.6383; geometry collision mesh filename=package://xarm_description/meshes/xarm7/visual/link3.stl; visual mesh filename=package://xarm_description/meshes/xarm7/visual/link3.stl
- link link4: mass 1.3192 -> 1.7269; geometry collision mesh filename=package://xarm_description/meshes/xarm7/visual/link4.stl; visual mesh filename=package://xarm_description/meshes/xarm7/visual/link4.stl
- link link5: mass 1.33854 -> 1.3203; geometry collision mesh filename=package://xarm_description/meshes/xarm7/visual/link5.stl; visual mesh filename=package://xarm_description/meshes/xarm7/visual/link5.stl
- link link6: mass 0.17 -> 1.325; geometry collision mesh filename=package://xarm_description/meshes/xarm7/visual/link6.stl; visual mesh filename=package://xarm_description/meshes/xarm7/visual/link6.stl
- link link_base: mass 2.7 -> 0.88556; geometry collision mesh filename=package://xarm_description/meshes/xarm7/visual/link_base.stl; visual mesh filename=package://xarm_description/meshes/xarm7/visual/link_base.stl
Joints:
- added joint joint7: type revolute, parent link6, child link7, origin xyz=0.076 0.097 0 rpy=-1.5708 0 0, axis 0 0 1, limit lower=-6.283185307179586 upper=6.283185307179586 effort=20 velocity=3.14
- joint joint1: limit lower=-6.283185307179586 upper=6.283185307179586 effort=50.0 velocity=3.14 -> lower=-6.283185307179586 upper=6.283185307179586 effort=50 velocity=3.14
- joint joint2: limit lower=-2.059 upper=2.0944 effort=50.0 velocity=3.14 -> lower=-2.059 upper=2.0944 effort=50 velocity=3.14
- joint joint3: limit lower=-3.927 upper=0.19198 effort=32.0 velocity=3.14 -> lower=-6.283185307179586 upper=6.283185307179586 effort=30 velocity=3.14; origin xyz=0.0535 -0.2845 0 rpy=0 0 0 -> xyz=0 -0.293 0 rpy=1.5708 0 0
- joint joint4: limit lower=-6.283185307179586 upper=6.283185307179586 effort=32.0 velocity=3.14 -> lower=-0.19198 upper=3.927 effort=30 velocity=3.14; origin xyz=0.0775 0.3425 0 rpy=-1.5708 0 0 -> xyz=0.0525 0 0 rpy=1.5708 0 0
- joint joint5: limit lower=-1.69297 upper=3.141592653589793 effort=32.0 velocity=3.14 -> lower=-6.283185307179586 upper=6.283185307179586 effort=30 velocity=3.14; origin xyz=0 0 0 rpy=1.5708 0 0 -> xyz=0.0775 -0.3425 0 rpy=1.5708 0 0
- joint joint6: limit lower=-6.283185307179586 upper=6.283185307179586 effort=20.0 velocity=3.14 -> lower=-1.69297 upper=3.141592653589793 effort=20 velocity=3.14; origin xyz=0.076 0.097 0 rpy=-1.5708 0 0 -> xyz=0 0 0 rpy=1.5708 0 0
- joint joint_eef: parent link6 -> link7
